File: kicad/usb_c.kicad_sch (KiCad schematic)
At the start: 22 parts, among them Q2 SS8050_C2150, Q3 SS8050_C2150, U4 CH343G

Commit message: Cleanups
Parts:
- C3, C5: LCSC C1525 -> (none)
- C4: LCSC C15849 -> (none)
- C6: LCSC C19702 -> (none)
- D6: LCSC C2290 -> (none); LCSC Part # (none) -> C2290
- D7: LCSC C72041 -> (none); LCSC Part # (none) -> C72041
- D8: LCSC C2286 -> (none); LCSC Part # (none) -> C2286
- D9: LCSC C72043 -> (none); LCSC Part # (none) -> C72043
- Q2, Q3: LCSC C2150 -> (none); LCSC Part C2150 -> (none); LCSC Part # (none) -> C2150
- R23, R24: LCSC C25752 -> (none); LCSC Part # (none) -> C25752
- R25, R26: LCSC C25905 -> (none); LCSC Part # (none) -> C25905
- R27, R28: LCSC C25744 -> (none); LCSC Part # (none) -> C25744
- R29, R30, R31, R32: LCSC C11702 -> (none); LCSC Part # (none) -> C11702
- U4: LCSC C2844153 -> (none); LCSC Part # (none) -> C2844153
- USBC1: LCSC C136423 -> (none); LCSC Part C136423 -> (none); LCSC Part # (none) -> C136423
Changed lines of the file:
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@@
       (effects (font (size 1.27 1.27)) hide)
     )
-    (property "LCSC" "C11702" (at 132.715 40.64 0)
+    (property "LCSC Part #" "C11702" (at 132.715 40.64 0)
       (effects (font (size 1.27 1.27)) hide)
     )
@@
       (effects (font (size 1.27 1.27)) hide)
     )
-    (property "LCSC" "C2286" (at 125.095 48.26 90)
+    (property "LCSC Part #" "C2286" (at 125.095 48.26 0)
       (effects (font (size 1.27 1.27)) hide)
     )
@@
       (effects (font (size 1.27 1.27)) hide)
     )
-    (property "LCSC" "C19702" (at 164.465 40.005 0)
-      (effects (font (size 1.27 1.27)) hide)
-    )
     (pin "1")
     (pin "2")
@@
       (effects (font (size 1.27 1.27)) hide)
     )
-    (property "LCSC" "C25744" (at 132.715 22.86 90)
+    (property "LCSC Part #" "C25744" (at 132.715 22.86 0)
       (effects (font (size 1.27 1.27)) hide)
     )
@@
       (effects (font (size 1.27 1.27)) hide)
     )
-    (property "LCSC" "C72043" (at 125.095 54.61 90)
+    (property "LCSC Part #" "C72043" (at 125.095 54.61 0)
       (effects (font (size 1.27 1.27)) hide)
     )
@@
       (effects (font (size 1.27 1.27)) hide)
     )
-    (property "LCSC" "C72041" (at 125.095 40.64 90)
+    (property "LCSC Part #" "C72041" (at 125.095 40.64 0)
       (effects (font (size 1.27 1.27)) hide)
     )
@@
       (effects (font (size 1.27 1.27)) hide)
     )
-    (property "LCSC" "C11702" (at 132.715 48.26 0)
+    (property "LCSC Part #" "C11702" (at 132.715 48.26 0)
       (effects (font (size 1.27 1.27)) hide)
     )
@@
       (effects (font (size 1.27 1.27)) hide)
     )
-    (property "LCSC" "C15849" (at 93.98 32.385 0)
-      (effects (font (size 1.27 1.27)) hide)
-    )
     (pin "1")
     (pin "2")
@@
       (effects (font (size 1.27 1.27)) hide)
     )
-    (property "LCSC" "C25744" (at 132.715 29.21 90)
+    (property "LCSC Part #" "C25744" (at 132.715 29.21 0)
       (effects (font (size 1.27 1.27)) hide)
     )
@@
       (effects (font (size 1.27 1.27)) hide)
     )
-    (property "LCSC" "C25752" (at 29.21 38.1 90)
+    (property "LCSC Part #" "C25752" (at 29.21 38.1 0)
       (effects (font (size 1.27 1.27)) hide)
     )
@@
       (effects (font (size 1.27 1.27)) hide)
     )
-    (property "LCSC" "C25752" (at 29.21 24.13 90)
+    (property "LCSC Part #" "C25752" (at 29.21 24.13 0)
       (effects (font (size 1.27 1.27)) hide)
     )
@@
       (effects (font (size 1.27 1.27)) hide)
     )
-    (property "LCSC" "C11702" (at 132.715 34.29 0)
+    (property "LCSC Part #" "C11702" (at 132.715 34.29 0)
       (effects (font (size 1.27 1.27)) hide)
     )
@@
       (effects (font (size 1.27 1.27)) hide)
     )
-    (property "LCSC" "C25905" (at 39.37 89.535 90)
+    (property "LCSC Part #" "C25905" (at 39.37 89.535 0)
       (effects (font (size 1.27 1.27)) hide)
     )
@@
       (effects (font (size 0 0)) hide)
     )
-    (property "LCSC Part" "C2150" (at 44.45 38.1 0)
-      (effects (font (size 0 0)) hide)
-    )
     (property "JLC Part" "Basic Part" (at 44.45 38.1 0)
       (effects (font (size 0 0)) hide)
     )
-    (property "LCSC" "C2150" (at 45.72 36.83 0)
+    (property "LCSC Part #" "C2150" (at 44.45 38.1 0)
       (effects (font (size 1.27 1.27)) hide)
     )
@@
       (effects (font (size 1.27 1.27)) hide)
     )
-    (property "LCSC" "C2290" (at 125.095 34.29 90)
+    (property "LCSC Part #" "C2290" (at 125.095 34.29 0)
       (effects (font (size 1.27 1.27)) hide)
     )
@@
     )
     (property "LCSC Part #" "C1525" (at 127 77.47 90)
-      (effects (font (size 1.27 1.27)) hide)
-    )
-    (property "LCSC" "C1525" (at 123.19 77.47 0)
       (effects (font (size 1.27 1.27)) hide)
     )
@@
       (effects (font (size 0 0)) hide)
     )
-    (property "LCSC Part" "C136423" (at 55.88 80.645 0)
-      (effects (font (size 0 0)) hide)
-    )
     (property "JLC Part" "Extended Part" (at 55.88 80.645 0)
       (effects (font (size 0 0)) hide)
     )
-    (property "LCSC" "C136423" (at 55.88 104.775 0)
+    (property "LCSC Part #" "C136423" (at 55.88 80.645 0)
       (effects (font (size 1.27 1.27)) hide)
     )
@@
       (effects (font (size 1.27 1.27)) hide)
     )
-    (property "LCSC" "C25905" (at 72.39 89.535 90)
+    (property "LCSC Part #" "C25905" (at 72.39 89.535 0)
       (effects (font (size 1.27 1.27)) hide)
     )
@@
       (effects (font (size 0 0)) hide)
     )
-    (property "LCSC Part" "C2150" (at 44.45 24.13 0)
-      (effects (font (size 0 0)) hide)
-    )
     (property "JLC Part" "Basic Part" (at 44.45 24.13 0)
       (effects (font (size 0 0)) hide)
     )
-    (property "LCSC" "C2150" (at 45.72 22.86 0)
+    (property "LCSC Part #" "C2150" (at 44.45 24.13 0)
       (effects (font (size 1.27 1.27)) hide)
     )
@@
       (effects (font (size 1.27 1.27)) hide)
     )
-    (property "LCSC" "C2844153" (at 109.22 96.52 0)
+    (property "LCSC Part #" "C2844153" (at 109.22 96.52 0)
       (effects (font (size 1.27 1.27)) hide)
     )
@@
       (effects (font (size 1.27 1.27)) hide)
     )
-    (property "LCSC" "C11702" (at 132.715 54.61 0)
+    (property "LCSC Part #" "C11702" (at 132.715 54.61 0)
       (effects (font (size 1.27 1.27)) hide)
     )
@@
       (effects (font (size 1.27 1.27)) hide)
     )
-    (property "LCSC" "C1525" (at 82.55 34.925 0)
-      (effects (font (size 1.27 1.27)) hide)
-    )
