File: kicad/boardcomputer-reinvented.kicad_sch (KiCad schematic)
At the start: 88 parts, among them J1 Conn_Display, J11 CAN1, J11 CAN2, J13 Conn_01x02_Pin, J14 Conn_01x05_Pin, J3 BREMSE, J3 GAS, J3 I2C, J5 Conn_01x02_Pin, J5 Conn_02x05_Odd_Even, J8 BREMSE, J8 GAS, Q1 2N7002, Q2 2N7002, U2 ESP32-S3-WROOM-1-ENTERTAINMENT, U2 SN65HVD231, U3 SHT30-DIS, U3 USBLC6-4SC6, U4 ESP32-S3-WROOM-1-CONTROL, U4 USBLC6-4SC6, U5 MPM2359, U6 USBLC6-4SC6, U7 USBLC6-4SC6, U8 USBLC6-4SC6

Commit message: Cleanups
Parts:
- removed J5 (x2): Conn_02x05_Odd_Even, Connector_PinHeader_2.54mm:PinHeader_2x05_P2.54mm_Vertical, symbol Connector_Generic:Conn_02x05_Odd_Even
- added C29: 100nF, Capacitor_SMD:C_0603_1608Metric, symbol Device:C
- added D6, D7: LED, LED_SMD:LED_0603_1608Metric, symbol Device:LED
- added J11: BUTTON3, Connector_JST:JST_XH_B5B-XH-A_1x05_P2.50mm_Vertical, symbol Connector_Generic:Conn_01x05
- added J11: BUTTON2, Connector_JST:JST_XH_B5B-XH-A_1x05_P2.50mm_Vertical, symbol Connector_Generic:Conn_01x05
- added J11: BUTTON1, Connector_JST:JST_XH_B5B-XH-A_1x05_P2.50mm_Vertical, symbol Connector_Generic:Conn_01x05
- added J11: BUTTON4, Connector_JST:JST_XH_B5B-XH-A_1x05_P2.50mm_Vertical, symbol Connector_Generic:Conn_01x05
- added J15: Conn_01x06_Pin, Connector_PinHeader_2.54mm:PinHeader_1x06_P2.54mm_Vertical, symbol Connector:Conn_01x06_Pin
- added JP3, JP4: SolderJumper_2_Open, Jumper:SolderJumper-2_P1.3mm_Open_RoundedPad1.0x1.5mm, symbol Jumper:SolderJumper_2_Open
- added R29, R30: 1k, Resistor_SMD:R_0402_1005Metric, symbol Device:R
- added R48, R49: 56, Resistor_SMD:R_0603_1608Metric, symbol Device:R
- added U3: USBLC6-4SC6, Package_TO_SOT_SMD:SOT-23-6, symbol Power_Protection:USBLC6-4SC6
- BZ1: footprint Smart Home Controller V3:Buzzer -> boardcomputer:Buzzer; LCSC C95299 -> (none); LCSC Part # (none) -> C95299
- C1: LCSC C19702 -> (none)
- C2: LCSC C1525 -> (none)
- C22: LCSC C1525 -> (none); LCSC Part # (none) -> C1525
- C4: LCSC C14663 -> (none); LCSC Part # (none) -> C14663
- D14: footprint Diode_SMD:D_SOD-123 -> Diode_SMD:D_SMB; symbol Device:D -> Diode:B230
- J3: LCSC C160404 -> (none); LCSC Part # (none) -> C160404
- Q1, Q2: LCSC C8545 -> (none); LCSC Part # (none) -> C8545
- R1, R15: LCSC C25744 -> (none); LCSC Part # (none) -> C25744
- R4, R5: LCSC C11702 -> (none); LCSC Part # (none) -> C11702
- R6, R7: LCSC C4190 -> (none); LCSC Part # (none) -> C4190
- U2, U4: footprint Espressif:ESP32-S3-WROOM-1 -> PCM_Espressif:ESP32-S3-WROOM-1; LCSC C2913199 -> (none); LCSC Part # (none) -> C2913199
- U3: LCSC C77361 -> (none); LCSC Part # (none) -> C77361
Connections:
- net +3V3: now also R29.1, R30.1, U3.5 (VBUS)
- net B1: now also J11.5 (Pin_5)
- net B10: now also J11.4 (Pin_4)
- net B11: now also J11.3 (Pin_3)
- net B12: now also J11.2 (Pin_2)
- net B13: now also J11.5 (Pin_5)
- net B14: now also J11.4 (Pin_4)
- net B15: now also J11.3 (Pin_3)
- net B16: now also J11.2 (Pin_2)
- net B2: now also J11.4 (Pin_4)
- net B3: now also J11.3 (Pin_3)
- net B4: now also J11.2 (Pin_2)
- net B5: now also J11.5 (Pin_5)
- net B6: now also J11.4 (Pin_4)
- net B7: now also J11.3 (Pin_3)
- net B8: now also J11.2 (Pin_2)
- net B9: now also J11.5 (Pin_5)
- net CANH: now also JP3.1 (A)
- net CANL: now also JP4.2 (B)
- net GND: now also C29.2, U3.2 (GND)
- net IN1: now also J11.1 (Pin_1); no longer U2.4 (GPIO4/TOUCH4/ADC1_CH3)
- net IN2: now also J11.1 (Pin_1); no longer U2.15 (GPIO3/TOUCH3/ADC1_CH2)
- net IN3: now also J11.1 (Pin_1); no longer U2.38 (GPIO2/TOUCH2/ADC1_CH1)
- net IN4: now also J11.1 (Pin_1); no longer U2.39 (GPIO1/TOUCH1/ADC1_CH0)
- net OUT1: no longer U2.5 (GPIO5/TOUCH5/ADC1_CH4)
- net OUT2: no longer U2.6 (GPIO6/TOUCH6/ADC1_CH5)
- net PROCESSOR_COMMUNICATION_CONTROLESP_RX: now also D7.1 (K), U3.6 (I/O4)
- net PROCESSOR_COMMUNICATION_CONTROLESP_TX: now also D6.1 (K), U3.4 (I/O3)
- new net: D6.2 (A), R29.2
- new net: D7.2 (A), R30.2
- new net: J15.4 (Pin_4), U2.15 (GPIO3/TOUCH3/ADC1_CH2)
- new net: J15.5 (Pin_5), U2.38 (GPIO2/TOUCH2/ADC1_CH1)
- new net: J15.6 (Pin_6), U2.39 (GPIO1/TOUCH1/ADC1_CH0)
- new net: J15.3 (Pin_3), U2.4 (GPIO4/TOUCH4/ADC1_CH3)
- new net: J15.2 (Pin_2), U2.5 (GPIO5/TOUCH5/ADC1_CH4)
- new net: J15.1 (Pin_1), U2.6 (GPIO6/TOUCH6/ADC1_CH5)
- new net: JP4.1 (A), R49.2
- new net: C29.1, R48.2, R49.1
- new net: JP3.2 (B), R48.1
- no-connect marks 28 -> 30
Other:
- moved on the sheet: D6

Commit message: Finished routing
Parts:
- removed J15: Conn_01x06_Pin, Connector_PinHeader_2.54mm:PinHeader_1x06_P2.54mm_Vertical, symbol Connector:Conn_01x06_Pin
- J1: footprint Connector_PinHeader_2.54mm:PinHeader_1x08_P2.54mm_Vertical -> Connector_PinHeader_2.54mm:PinHeader_2x04_P2.54mm_Vertical
- J13: footprint Connector_Wire:SolderWire-2sqmm_1x02_P7.8mm_D2mm_OD3.9mm -> Connector_Wire:SolderWire-1sqmm_1x02_P5.4mm_D1.4mm_OD2.7mm
- J5: footprint Connector_AMASS:AMASS_XT30PW-M_1x02_P2.50mm_Horizontal -> Connector_Wire:SolderWire-1sqmm_1x02_P5.4mm_D1.4mm_OD2.7mm; LCSC Part # C431092 -> (none)
Connections:
- net RAW_M365_BREMS is gone; now on net RAW_M365_BREMSE: U4.39 (GPIO1/TOUCH1/ADC1_CH0), U8.6 (I/O4)
- net +3.3V: now also C4.1, C4.1, C4.1, J3.2 (Pin_2), J3.3 (Pin_3), J3.3 (Pin_3), J8.3 (Pin_3), J8.3 (Pin_3), R29.1, R30.1, R5.1, R5.1, R5.1, R5.1, R6.2, R7.2, U2.3 (VCC), U2.3 (VCC), U3.5 (VBUS), U3.5 (VBUS), U3.5 (VDD), U4.5 (VBUS), U6.5 (VBUS), U7.5 (VBUS), U8.5 (VBUS)
- net B10: now also D7.2 (A); no longer D10.2 (A)
- net B11: now also D9.1 (K); no longer D11.1 (K)
- net B12: now also D9.2 (A); no longer D11.2 (A)
- net B13: now also D11.1 (K); no longer D12.1 (K)
- net B14: now also D11.2 (A); no longer D12.2 (A)
- net B3: now also D8.1 (K); no longer D7.1 (K)
- net B4: now also D8.2 (A); no longer D7.2 (A)
- net B5: now also D10.1 (K); no longer D8.1 (K)
- net B6: now also D10.2 (A); no longer D8.2 (A)
- net B7: now also D12.1 (K); no longer D9.1 (K)
- net B8: now also D12.2 (A); no longer D9.2 (A)
- net B9: now also D7.1 (K); no longer D10.1 (K)
- net GND: now also J13.1 (Pin_1), J3.1 (Pin_1), J3.1 (Pin_1), J8.1 (Pin_1), J8.1 (Pin_1); no longer J13.2 (Pin_2), J3.3 (Pin_3), J3.3 (Pin_3), J8.3 (Pin_3), J8.3 (Pin_3)
- net at D6.2 (A), J5.2 (Pin_2): now also J13.2 (Pin_2); no longer J13.1 (Pin_1)
- removed net +3V3: C4.1, C4.1, C4.1, J3.1 (Pin_1), J3.1 (Pin_1), J3.2 (Pin_2), J8.1 (Pin_1), J8.1 (Pin_1), R29.1, R30.1, R5.1, R5.1, R5.1, R5.1, R6.2, R7.2, U2.3 (VCC), U2.3 (VCC), U3.5 (VBUS), U3.5 (VBUS), U3.5 (VDD), U4.5 (VBUS), U6.5 (VBUS), U7.5 (VBUS), U8.5 (VBUS)
Other:
- moved on the sheet: J13

Commit message: Updated pcb
Parts:
- removed C22: 100n, Capacitor_SMD:C_0402_1005Metric, symbol Device:C_Small
- removed R13 (x2): 100k, Resistor_SMD:R_0603_1608Metric, symbol Device:R
- removed R5 (x2): 10k, Resistor_SMD:R_0402_1005Metric, symbol Device:R
- removed R5 (x2): 1k, Resistor_SMD:R_0402_1005Metric, symbol Device:R
- added R5 (x4): 10k, Resistor_SMD:R_0402_1005Metric, symbol Device:R
- J3, J8: footprint Connector_PinHeader_2.54mm:PinHeader_1x03_P2.54mm_Vertical -> Connector_JST:JST_XH_B3B-XH-A_1x03_P2.50mm_Vertical; LCSC Part # DNP -> C144394
Connections:
- net +3.3V: now also R5.2, R5.2
- net B10: now also J11.2 (Pin_2), U3.4 (I/O3); no longer J11.4 (Pin_4), U6.3 (I/O2)
- net B13: now also J11.3 (Pin_3), U4.6 (I/O4); no longer J11.5 (Pin_5), U7.1 (I/O1)
- net B14: now also J11.2 (Pin_2), U4.4 (I/O3); no longer J11.4 (Pin_4), U7.3 (I/O2)
- net B3: now also J11.5 (Pin_5), U6.3 (I/O2); no longer J11.3 (Pin_3), U3.4 (I/O3)
- net B4: now also J11.4 (Pin_4), U6.1 (I/O1); no longer J11.2 (Pin_2), U3.6 (I/O4)
- net B7: now also J11.5 (Pin_5), U7.3 (I/O2); no longer J11.3 (Pin_3), U4.4 (I/O3)
- net B8: now also J11.4 (Pin_4), U7.1 (I/O1); no longer J11.2 (Pin_2), U4.6 (I/O4)
- net B9: now also J11.3 (Pin_3), U3.6 (I/O4); no longer J11.5 (Pin_5), U6.1 (I/O1)
- net CONTROLESP_CAN_RX: now also R5.2
- net CONTROLESP_CAN_TX: now also R5.1
- net ENTERTAINMENT_CAN_RX: now also R5.2
- net ENTERTAINMENT_CAN_TX: now also R5.1
- net GND: now also R5.1, R5.1
